File: LIS3DH-breakout.kicad_pcb (KiCad board)
At the start: 2 copper layers, 21.8 x 26 mm, 15 parts, among them J1 Conn_01x06_Female, J2 Conn_01x06_Female

Commit message: added logo
Parts:
- added G***: LOGO, LOGO, B.Cu at (141.5, 104.4)
Other:
- board text added: "LIS3DH Breakout board, v1 Jed Parsons github.com/jedp/"
